File: electrical/motion_control/board/board.kicad_pcb (KiCad board)
At the start: 4 copper layers, 106 x 98 mm, 64 parts, among them J101 5V_IN, J201 I2C_Socket, J202 ETH, J203 Debug_Socket, J301 USB_MASKROM, J401 USB_1, J402 USB_0, J403 RS485_0, J404 RS485_1, J601 SPI00_CAN_OUT, J602 SPI01_CAN_OUT, J603 SPI02_CAN_OUT, J701 CAN0_OUT, J702 CAN1_OUT, J703 CAN2_OUT, U101 AMS1117-3.3, U201 Hirose DF40C-100DS-0.4V, U202 LSM6DSVTR, U301 Hirose DF40C-100DS-0.4V, U401 Hirose DF40C-100DS-0.4V, U402 SN65HVD10DR, U403 TXB0104PW, U404 TXB0104PW, U405 SN65HVD10DR, U501 MCP2518FD-xQBB, U502 MCP2518FD-xQBB, U503 MCP2518FD-xQBB, U602 TXB0104PW, U603 SN65HVD230, U606 SN65HVD230, U607 SN65HVD230, U701 SN65HVD230, U702 SN65HVD230, U703 SN65HVD230, Y601 40M, Y602 40M, Y603 40M

Commit message: new boards, new device tree image
Parts:
- removed C401, C402, C403, C404: 100n, Capacitor_SMD:C_0402_1005Metric
- removed the C603 at (114.4, 91.8)
- removed J201: I2C_Socket, Connector_JST:JST_GH_SM04B-GHS-TB_1x04-1MP_P1.25mm_Horizontal
- removed J202: ETH, Connector_JST:JST_GH_BM08B-GHS-TBT_1x08-1MP_P1.25mm_Vertical
- removed J203: Debug_Socket, Connector_JST:JST_GH_SM04B-GHS-TB_1x04-1MP_P1.25mm_Horizontal
- removed J301: USB_MASKROM, Connector_JST:JST_GH_SM04B-GHS-TB_1x04-1MP_P1.25mm_Horizontal
- removed J401: USB_1, Connector_JST:JST_GH_SM04B-GHS-TB_1x04-1MP_P1.25mm_Horizontal
- removed J402: USB_0, Connector_JST:JST_GH_SM04B-GHS-TB_1x04-1MP_P1.25mm_Horizontal
- removed J403: RS485_0, Connector_JST:JST_GH_SM02B-GHS-TB_1x02-1MP_P1.25mm_Horizontal
- removed J404: RS485_1, Connector_JST:JST_GH_SM02B-GHS-TB_1x02-1MP_P1.25mm_Horizontal
- removed J601: SPI00_CAN_OUT, Connector_JST:JST_GH_SM02B-GHS-TB_1x02-1MP_P1.25mm_Horizontal
- removed J602: SPI01_CAN_OUT, Connector_JST:JST_GH_SM02B-GHS-TB_1x02-1MP_P1.25mm_Horizontal
- removed J603: SPI02_CAN_OUT, Connector_JST:JST_GH_SM02B-GHS-TB_1x02-1MP_P1.25mm_Horizontal
- removed J701: CAN0_OUT, Connector_JST:JST_GH_SM02B-GHS-TB_1x02-1MP_P1.25mm_Horizontal
- removed J702: CAN1_OUT, Connector_JST:JST_GH_SM02B-GHS-TB_1x02-1MP_P1.25mm_Horizontal
- removed J703: CAN2_OUT, Connector_JST:JST_GH_SM02B-GHS-TB_1x02-1MP_P1.25mm_Horizontal
- removed R401, R402: 10k, Resistor_SMD:R_0402_1005Metric
- removed the R602 at (109.1, 82.8)
- removed R701, R702, R703: 120, Resistor_SMD:R_0402_1005Metric
- removed TP201, TP202, TP203, TP401: TestPoint, TestPoint:TestPoint_Pad_D1.0mm
- removed U402, U405: SN65HVD10DR, lcsc_lib:SOIC-8_L4.9-W3.9-P1.27-LS6.0-BL
- removed U403, U404: TXB0104PW, Package_SO:TSSOP-14_4.4x5mm_P0.65mm
- removed the U602 at (111.8, 87.3)
- removed U703: SN65HVD230, Package_SO:SOIC-8_3.9x4.9mm_P1.27mm
- added C101: 4.7u, Capacitor_SMD:C_0402_1005Metric, F.Cu at (116.8, 128.8)
- added C102: 1n, Capacitor_SMD:C_0402_1005Metric, F.Cu at (116.8, 130.9)
- added C103: 4.7u, Capacitor_SMD:C_0402_1005Metric, F.Cu at (122.4, 128.8)
- added C203: 1n, Capacitor_SMD:C_1206_3216Metric, F.Cu at (150.5, 46.5)
- added C204: 100n, Capacitor_SMD:C_0402_1005Metric, F.Cu at (139.2, 60.0)
- added C205: 100n, Capacitor_SMD:C_0402_1005Metric, F.Cu at (137.5, 60.0)
- added C501: 100n, Capacitor_SMD:C_0402_1005Metric, B.Cu at (166.0, 110.0)
- added C502: 100n, Capacitor_SMD:C_0402_1005Metric, B.Cu at (173.2, 109.8)
- added C503: 100n, Capacitor_SMD:C_0402_1005Metric, B.Cu at (116.0, 78.5)
- added C504: 100n, Capacitor_SMD:C_0402_1005Metric, B.Cu at (115.8, 71.4)
- added C505: 100n, Capacitor_SMD:C_0402_1005Metric, B.Cu at (115.2, 111.0)
- added C506: 100n, Capacitor_SMD:C_0402_1005Metric, B.Cu at (108.8, 113.0)
- added C507: 100n, Capacitor_SMD:C_0402_1005Metric, B.Cu at (115.2, 103.5)
- added C508: 100n, Capacitor_SMD:C_0402_1005Metric, B.Cu at (108.8, 120.5)
- added C601: 20p, Capacitor_SMD:C_0603_1608Metric, B.Cu at (102.6, 123.3)
- added C608: 20p, Capacitor_SMD:C_0603_1608Metric, B.Cu at (116.2, 81.8)
- added C609: 20p, Capacitor_SMD:C_0603_1608Metric, B.Cu at (140.5, 119.8)
- added C611: 20p, Capacitor_SMD:C_0603_1608Metric, B.Cu at (110.7, 81.8)
- added C612: 20p, Capacitor_SMD:C_0603_1608Metric, B.Cu at (140.5, 125.2)
- added G***: LOGO, LOGO, B.Cu at (138.4, 67.9)
- added J102: HEADER_BOTTOM, Connector_PinHeader_2.54mm:PinHeader_2x08_P2.54mm_Vertical, F.Cu at (129.5, 133.0)
- added J103: HEADER_RIGHT, Connector_PinHeader_2.54mm:PinHeader_2x08_P2.54mm_Vertical, F.Cu at (178.9, 81.0)
- added R201: 1M, Resistor_SMD:R_2010_5025Metric, F.Cu at (150.5, 52.5)
- added R202: 100, Resistor_SMD:R_0402_1005Metric, F.Cu at (156.7, 129.5)
- added R301: 5.1k, Resistor_SMD:R_0402_1005Metric, F.Cu at (167.1, 125.3)
- added R302: 5.1k, Resistor_SMD:R_0402_1005Metric, F.Cu at (170.3, 125.3)
- added R501: 10k, Resistor_SMD:R_0402_1005Metric, B.Cu at (173.2, 103.2)
- added R502: 10k, Resistor_SMD:R_0402_1005Metric, B.Cu at (109.3, 71.4)
- added R503: 10k, Resistor_SMD:R_0402_1005Metric, B.Cu at (108.8, 103.5)
- added R504: 10k, Resistor_SMD:R_0402_1005Metric, B.Cu at (115.2, 120.5)
- added R601: 120, Resistor_SMD:R_0402_1005Metric, F.Cu at (100.8, 118.5)
- added R605: 120, Resistor_SMD:R_0402_1005Metric, F.Cu at (100.8, 89.0)
- added R606: 120, Resistor_SMD:R_0402_1005Metric, F.Cu at (153.5, 127.0)
- added SW201: TS50810-411-02528, lcsc_lib:SW-SMD_L6.2-W3.7-LS8.0, F.Cu at (156.8, 132.2)
- added U202: ETH, lcsc_lib:RJ45-SMD_HR963380AE, F.Cu at (138.4, 47.9)
- added U501: TXB0104PW, Package_SO:TSSOP-14_4.4x5mm_P0.65mm, B.Cu at (169.5, 106.5)
- added U502: TXB0104PW, Package_SO:TSSOP-14_4.4x5mm_P0.65mm, B.Cu at (112.6, 75.1)
- added U503: TXB0104PW, Package_SO:TSSOP-14_4.4x5mm_P0.65mm, B.Cu at (112.1, 107.2)
- added U504: TXB0104PW, Package_SO:TSSOP-14_4.4x5mm_P0.65mm, B.Cu at (112.0, 116.8)
- added U601: MCP2518FD-xQBB, Package_SO:SOIC-14_3.9x8.7mm_P1.27mm, B.Cu at (109.0, 127.5)
- added U604: SN65HVD230, Package_SO:SOIC-8_3.9x4.9mm_P1.27mm, F.Cu at (104.2, 118.5)
- added U608: MCP2518FD-xQBB, Package_SO:SOIC-14_3.9x8.7mm_P1.27mm, B.Cu at (113.8, 88.0)
- added U609: MCP2518FD-xQBB, Package_SO:SOIC-14_3.9x8.7mm_P1.27mm, B.Cu at (146.5, 123.2)
- added U611: SN65HVD230, Package_SO:SOIC-8_3.9x4.9mm_P1.27mm, F.Cu at (104.2, 89.2)
- added U612: SN65HVD230, Package_SO:SOIC-8_3.9x4.9mm_P1.27mm, F.Cu at (153.5, 122.5)
- added USB301: TYPE-C 16PIN 2MD, lcsc_lib:USB-C-SMD_TYPE-C-16PIN-2MD-073, F.Cu at (168.5, 129.7)
- added Y601: 40M, Crystal:Crystal_SMD_3225-4Pin_3.2x2.5mm, B.Cu at (102.7, 126.0)
- added Y605: 40M, Crystal:Crystal_SMD_3225-4Pin_3.2x2.5mm, B.Cu at (113.5, 81.8)
- added Y606: 40M, Crystal:Crystal_SMD_3225-4Pin_3.2x2.5mm, B.Cu at (140.5, 122.5)
- C602: renamed from C601; moved to B.Cu
- C603: renamed from C606; moved to B.Cu
- C604: value 100n -> 20p; footprint Capacitor_SMD:C_0402_1005Metric -> Capacitor_SMD:C_0603_1608Metric
- C605: renamed from C602; moved to B.Cu
- C606: renamed from C608; moved to B.Cu
- C607: renamed from C605; moved to B.Cu
- C610: renamed from C607; moved to B.Cu
- J101: value 5V_IN -> HEADER_LEFT; footprint Connector_AMASS:AMASS_XT30UPB-F_1x02_P5.0mm_Vertical -> Connector_PinHeader_2.54mm:PinHeader_2x08_P2.54mm_Vertical
- U101: value AMS1117-3.3 -> ADM7172ACPZ-3.3-R7; footprint Package_TO_SOT_SMD:SOT-223-3_TabPin2 -> lcsc_lib:DFN-8_L3.0-W3.0-P0.50-BL-EP
- U602: renamed from U501; moved to B.Cu
- U603: renamed from U503; moved to B.Cu
- U607: renamed from U502; moved to B.Cu
- U701, U702: value SN65HVD230 -> SN65HVD10DR; footprint Package_SO:SOIC-8_3.9x4.9mm_P1.27mm -> lcsc_lib:SOIC-8_L4.9-W3.9-P1.27-LS6.0-BL
- Y602: renamed from Y601; moved to B.Cu
- Y603: moved to B.Cu
- Y604: renamed from Y602; moved to B.Cu
- moved J101 55.2 mm to (95.3, 81.0), turned to 0 degrees
- moved C606 51.7 mm to (107.4, 97.0), turned to 180 degrees
- moved Y603 48.3 mm to (107.4, 94.3), turned to 0 degrees
- moved C604 47.4 mm to (102.6, 128.8), turned to 180 degrees
- moved C603 45.0 mm to (107.4, 91.6), turned to 0 degrees
- moved U606 44.5 mm to (104.2, 97.5), turned to -90 degrees
- moved U603 43.8 mm to (113.8, 96.9), turned to 0 degrees
- moved R603 43.7 mm to (100.8, 97.0), turned to -90 degrees
- moved U702 26.6 mm to (104.2, 111.5), turned to 90 degrees
- moved C607 25.2 mm to (116.9, 49.1), turned to -90 degrees
- moved Y604 21.6 mm to (114.1, 49.0), turned to -90 degrees
- moved C602 20.4 mm to (106.6, 61.0)
- moved C610 17.9 mm to (111.3, 49.0), turned to 90 degrees
- moved Y602 15.0 mm to (106.5, 63.7)
- moved U610 13.9 mm to (104.2, 72.8), turned to -90 degrees
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- renumbered R601 to R602, R605 to R603, U202 to U203, U603 to U605, U607 to U606, U606 to U610
Connections:
- net /J1/SPI0_CS2 renamed /J1/SPI1_CS0
- net /J1/SPI0_INT2 renamed /J1/SPI1_INT0
- net /SPI-CAN/SPI02_OSC_1 renamed /SPI-CAN/SPI10_OSC_1
- net /SPI-CAN/SPI02_OSC_2 renamed /SPI-CAN/SPI10_OSC_2
- C604 pad 1: +3V3 -> /SPI-CAN/SPI40_OSC_2
- J101 pad 1: GND -> CAN0+
- J101 pad 2: +5V -> CAN3+
- R602 pad 1: /SPI-CAN/SPI00_CAN+ -> CAN3+
- R602 pad 2: /SPI-CAN/SPI00_CAN- -> CAN3-
- R603 pad 1: /SPI-CAN/SPI02_CAN+ -> CAN4+
- R603 pad 2: /SPI-CAN/SPI02_CAN- -> CAN4-
- R604 pad 1: /SPI-CAN/SPI01_CAN+ -> CAN0+
- R604 pad 2: /SPI-CAN/SPI01_CAN- -> CAN0-
- U101 pad 1: GND -> +3V3
- U101 pad 3: +5V -> +3V3
- U201 pad 21: /CAN/TXCAN1 -> unconnected-(U201-PI_nLED_Activity-Pad21)
- U201 pad 24: unconnected-(U201-GPIO26-Pad24) -> /RS485/UART4_RX_M1
- U201 pad 31: /CAN/RXCAN1 -> unconnected-(U201-GPIO12-Pad31)
- U201 pad 34: /J1/UART4_CTSN_1V8 -> unconnected-(U201-GPIO5-Pad34)
- U201 pad 38: /SPI-CAN/SPI0_CLK_M2_1V8 -> /TTL-SHIFT/SPI0_CLK_M2_1V8
- U201 pad 40: /SPI-CAN/SPI0_MISO_M2_1V8 -> /TTL-SHIFT/SPI0_MISO_M2_1V8
- U201 pad 44: /SPI-CAN/SPI0_MOSI_M2_1V8 -> /TTL-SHIFT/SPI0_MOSI_M2_1V8
- U201 pad 46: /J1/UART3_CTSN_1V8 -> unconnected-(U201-GPIO22-Pad46)
- U201 pad 48: /J1/UART4_RTSN_1V8 -> /TTL-SHIFT/UART4_RTSN_1V8
- U201 pad 50: /J1/UART3_RTSN_1V8 -> /TTL-SHIFT/SPI4_CLK_M0_1V8
- U201 pad 51: /U13A/UART2_RX_M0 -> UART2_RX_M0
- U201 pad 55: /U13A/UART2_TX_M0 -> UART2_TX_M0
- U201 pad 57: /CAN/RXCAN0 -> unconnected-(U201-SD_CLK-Pad57)
- U201 pad 61: /U13A/I2C8_SDA_M0 -> unconnected-(U201-SD_DAT3-Pad61)
- U201 pad 62: /CAN/TXCAN0 -> unconnected-(U201-SD_CMD-Pad62)
- U201 pad 69: /U13A/I2C8_SCL_M0 -> unconnected-(U201-SD_DAT2-Pad69)
- U201 pad 89: unconnected-(U201-WiFi_nDisable-Pad89) -> /RS485/UART0_TX_M0
- U201 pad 91: unconnected-(U201-BT_nDisable-Pad91) -> /RS485/UART0_RTSN
- U301 pad 109: unconnected-(U301-PCIe_nRST-Pad109) -> /RS485/UART4_TX_M1
- U401 pad 204: unconnected-(U401-GPIO_3V3_1-Pad204) -> /J1/GPIO3_C0_3V3
- U401 pad 206: unconnected-(U401-GPIO_3V3_2-Pad206) -> /J1/GPIO3_B7_3V3
- U401 pad 208: unconnected-(U401-GPIO_3V3_3-Pad208) -> /J1/GPIO3_C4_3V3
- U401 pad 214: unconnected-(U401-GPIO_3V3_4-Pad214) -> /J1/GPIO3_D4_3V3
- U401 pad 220: /J1/UART3_TX_M0_1V8 -> /J1/SPI4_MOSI_M0_1V8
- U401 pad 224: /J1/UART4_RX_M0_1V8 -> unconnected-(U401-GPIO_1V8_4-Pad224)
- U401 pad 236: /J1/UART3_RX_M0_1V8 -> /J1/SPI4_MISO_M0_1V8
- U401 pad 244: unconnected-(U401-GPIO_1V8_6-Pad244) -> /J1/SPI1_MISO_M2_1V8
- U401 pad 245: /J1/USB2_HOST1_D+ -> USB2_HOST0_D-
- U401 pad 246: unconnected-(U401-GPIO_1V8_7-Pad246) -> /J1/SPI1_MOSI_M2_1V8
- U401 pad 247: /J1/USB2_HOST1_D- -> USB2_HOST0_D+
- U401 pad 263: /J1/USB2_HOST0_D+ -> USB2_HOST1_D-
- U401 pad 265: /J1/USB2_HOST0_D- -> USB2_HOST1_D+
- U401 pad 283: /J1/UART4_TX_M0_1V8 -> /J1/SPI1_CLK_M2_1V8
- U401 pad 285: unconnected-(U401-GPIO_3V3_12-Pad285) -> /J1/SPI4_INT0
- U401 pad 287: unconnected-(U401-GPIO_3V3_13-Pad287) -> /J1/SPI4_CS0
- U401 pad 289: unconnected-(U401-GPIO_3V3_14-Pad289) -> /J1/SPI4_INT1
- U401 pad 293: unconnected-(U401-GPIO_3V3_15-Pad293) -> /J1/SPI4_CS1
- U401 pad 294: unconnected-(U401-GPIO_3V3_9-Pad294) -> /J1/SPI1_CS1
- U401 pad 295: /CAN/TXCAN2 -> unconnected-(U401-TYPEC5V_PWREN_H-Pad295)
- U401 pad 296: unconnected-(U401-GPIO_3V3_CC_INT0_L-Pad296) -> /J1/UART0_RX_M0
- U401 pad 298: /CAN/RXCAN2 -> /J1/SPI1_INT1
- U603 pad 10: /SPI-CAN/SPI0_CLK -> /SPI-CAN/SPI1_CLK
- U603 pad 11: /SPI-CAN/SPI0_SI -> /SPI-CAN/SPI1_SI
- U603 pad 12: /SPI-CAN/SPI0_SO -> /SPI-CAN/SPI1_SO
- U605 pad 6: /SPI-CAN/SPI00_CAN- -> CAN3-
- U605 pad 7: /SPI-CAN/SPI00_CAN+ -> CAN3+
- U606 pad 6: /SPI-CAN/SPI02_CAN- -> CAN4-
- U606 pad 7: /SPI-CAN/SPI02_CAN+ -> CAN4+
- U610 pad 6: /SPI-CAN/SPI01_CAN- -> CAN0-
- U610 pad 7: /SPI-CAN/SPI01_CAN+ -> CAN0+
- U701 pad 1: /CAN/TXCAN0 -> /RS485/UART4_RX_M1
- U701 pad 2: GND -> /RS485/UART4_RTSN
- U701 pad 3: +3V3 -> /RS485/UART4_RTSN
- U701 pad 4: /CAN/RXCAN0 -> /RS485/UART4_TX_M1
- U701 pad 5: unconnected-(U701-Vref-Pad5) -> GND
- U701 pad 6: /CAN/CAN0- -> RS0+
- U701 pad 7: /CAN/CAN0+ -> RS0-
- U701 pad 8: GND -> +3V3
- U702 pad 1: /CAN/TXCAN1 -> /J1/UART0_RX_M0
- U702 pad 2: GND -> /RS485/UART0_RTSN
- U702 pad 3: +3V3 -> /RS485/UART0_RTSN
- U702 pad 4: /CAN/RXCAN1 -> /RS485/UART0_TX_M0
- U702 pad 5: unconnected-(U702-Vref-Pad5) -> GND
- U702 pad 6: /CAN/CAN1- -> RS1+
- U702 pad 7: /CAN/CAN1+ -> RS1-
- U702 pad 8: GND -> +3V3
Routing:
- net /J1/SPI1_CS0: track 108.0 -> 35.4 mm
- net /U13A/UART2_RX_M0: track 69.5 -> 0.00 mm, vias 2 -> 0
- net /U13A/UART2_TX_M0: track 69.2 -> 0.00 mm, vias 2 -> 0
- net /U13B/USB2_D+: track 30.4 -> 99.2 mm
- net /U13B/USB2_D-: track 30.4 -> 99.1 mm
- net UART2_TX_M0: track 0.00 -> 64.6 mm, vias 0 -> 1
- net UART2_RX_M0: track 0.00 -> 64.6 mm, vias 0 -> 1
- net /J1/SPI1_INT0: track 103.2 -> 38.6 mm
- net /RS485/UART4_TX_M1: track 0.00 -> 57.5 mm, vias 0 -> 3
- net /SPI-CAN/SPI4_CLK: track 0.00 -> 57.4 mm
- net /SPI-CAN/SPI4_SO: track 0.00 -> 57.1 mm
- net /SPI-CAN/SPI4_SI: track 0.00 -> 56.9 mm
- net /J1/GPIO3_C0_3V3: track 0.00 -> 55.0 mm, vias 0 -> 2
- net USB2_HOST0_D-: track 0.00 -> 54.1 mm
- net USB2_HOST0_D+: track 0.00 -> 54.1 mm
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- added copper zone on F.Cu, net +5V
- removed copper zone on F.Cu, net GND
Other:
- board text added: "ASV1_100 MCB-V1.1"
- board text added: "ENGINEERED BY MENLO RESEARCH"
- board text removed: "C0"
- board text removed: "C1"
- board text removed: "C2"
- board text removed: "C3"
- board text removed: "C4"
- board text removed: "C5"
- board text removed: "DBG"
- board text removed: "I2C"
- board text removed: "MCB-V0.1.4"
- board text removed: "R0"
- board text removed: "R1"
- board text removed: "U0"
- board text removed: "U1"
- board text removed: "U2"
