File: electrical/motion_control/board/can.kicad_sch (KiCad schematic)
At the start: 9 parts, among them J701 CAN0_OUT, J702 CAN1_OUT, J703 CAN2_OUT, U701 SN65HVD230, U702 SN65HVD230, U703 SN65HVD230

Commit message: new boards, new device tree image
Parts:
- removed J701: CAN0_OUT, Connector_JST:JST_GH_SM02B-GHS-TB_1x02-1MP_P1.25mm_Horizontal, symbol Connector:Conn_01x02_Pin
- removed J702: CAN1_OUT, Connector_JST:JST_GH_SM02B-GHS-TB_1x02-1MP_P1.25mm_Horizontal, symbol Connector:Conn_01x02_Pin
- removed J703: CAN2_OUT, Connector_JST:JST_GH_SM02B-GHS-TB_1x02-1MP_P1.25mm_Horizontal, symbol Connector:Conn_01x02_Pin
- removed R701, R702, R703: 120, Resistor_SMD:R_0402_1005Metric, symbol Device:R_Small
- removed U701, U702, U703: SN65HVD230, Package_SO:SOIC-8_3.9x4.9mm_P1.27mm, symbol Interface_CAN_LIN:SN65HVD230
Connections:
- no-connect marks 3 -> 0
