File: electrical/motion_control/board/cm5-j1.kicad_sch (KiCad schematic)
At the start: 16 parts, among them J401 USB_1, J402 USB_0, J403 RS485_0, J404 RS485_1, U401 Hirose DF40C-100DS-0.4V, U402 SN65HVD10DR, U403 TXB0104PW, U404 TXB0104PW, U405 SN65HVD10DR

Commit message: new boards, new device tree image
Parts:
- removed C401, C402, C403, C404: 100n, Capacitor_SMD:C_0402_1005Metric, symbol Device:C_Small
- removed J401: USB_1, Connector_JST:JST_GH_SM04B-GHS-TB_1x04-1MP_P1.25mm_Horizontal, symbol Connector:Conn_01x04_Socket
- removed J402: USB_0, Connector_JST:JST_GH_SM04B-GHS-TB_1x04-1MP_P1.25mm_Horizontal, symbol Connector:Conn_01x04_Socket
- removed J403: RS485_0, Connector_JST:JST_GH_SM02B-GHS-TB_1x02-1MP_P1.25mm_Horizontal, symbol Connector:Conn_01x02_Pin
- removed J404: RS485_1, Connector_JST:JST_GH_SM02B-GHS-TB_1x02-1MP_P1.25mm_Horizontal, symbol Connector:Conn_01x02_Pin
- removed R401, R402: 10k, Resistor_SMD:R_0402_1005Metric, symbol Device:R_Small
- removed TP401: TestPoint, TestPoint:TestPoint_Pad_D1.0mm, symbol Connector:TestPoint
- removed U402, U405: SN65HVD10DR, lcsc_lib:SOIC-8_L4.9-W3.9-P1.27-LS6.0-BL, symbol lcsc_lib:SN65HVD10DR
- removed U403, U404: TXB0104PW, Package_SO:TSSOP-14_4.4x5mm_P0.65mm, symbol Logic_LevelTranslator:TXB0104PW
Connections:
- net USB2_HOST0_D+: now also U401.247 (USB3_HOST1_DM); no longer U401.263 (USB2_HOST2_DP)
- net USB2_HOST0_D-: now also U401.245 (USB3_HOST1_DP); no longer U401.265 (USB2_HOST2_DM)
- net USB2_HOST1_D+: now also U401.265 (USB2_HOST2_DM); no longer U401.245 (USB3_HOST1_DP)
- net USB2_HOST1_D-: now also U401.263 (USB2_HOST2_DP); no longer U401.247 (USB3_HOST1_DM)
- net GPIO3_C0_3V3: now reaches U401.204 (GPIO_3V3_1)
- net GPIO3_B7_3V3: now reaches U401.206 (GPIO_3V3_2)
- net GPIO3_C4_3V3: now reaches U401.208 (GPIO_3V3_3)
- net GPIO3_D4_3V3: now reaches U401.214 (GPIO_3V3_4)
- net SPI1_MISO_M2_1V8: now reaches U401.244 (GPIO_1V8_6)
- net SPI1_MOSI_M2_1V8: now reaches U401.246 (GPIO_1V8_7)
- net SPI4_INT0: now reaches U401.285 (GPIO_3V3_12)
- net SPI4_CS0: now reaches U401.287 (GPIO_3V3_13)
- net SPI4_INT1: now reaches U401.289 (GPIO_3V3_14)
- net SPI4_CS1: now reaches U401.293 (GPIO_3V3_15)
- net SPI1_CS1: now reaches U401.294 (GPIO_3V3_9)
- net UART0_RX_M0: now reaches U401.296 (GPIO_3V3_CC_INT0_L)
- net CAN2_RX_M1 renamed SPI1_INT1
- net CAN2_TX_M1: no longer names the net of U401.295 (TYPEC5V_PWREN_H)
- net SPI0_CS2 renamed SPI1_CS0
- net SPI0_INT2 renamed SPI1_INT0
- net UART3_RX_M0_1V8 renamed SPI4_MISO_M0_1V8
- net UART3_TX_M0_1V8 renamed SPI4_MOSI_M0_1V8
- net UART4_RX_M0_1V8: no longer names the net of U401.224 (GPIO_1V8_4)
- net UART4_TX_M0_1V8 renamed SPI1_CLK_M2_1V8
- no-connect marks 44 -> 34
