File: electrical/motion_control/board/cm5-u13a.kicad_sch (KiCad schematic)
At the start: 10 parts, among them J201 I2C_Socket, J202 ETH, J203 Debug_Socket, U201 Hirose DF40C-100DS-0.4V, U202 LSM6DSVTR

Commit message: new boards, new device tree image
Parts:
- removed J201: I2C_Socket, Connector_JST:JST_GH_SM04B-GHS-TB_1x04-1MP_P1.25mm_Horizontal, symbol Connector:Conn_01x04_Socket
- removed J202: ETH, Connector_JST:JST_GH_BM08B-GHS-TBT_1x08-1MP_P1.25mm_Vertical, symbol Connector_Generic:Conn_01x08
- removed J203: Debug_Socket, Connector_JST:JST_GH_SM04B-GHS-TB_1x04-1MP_P1.25mm_Horizontal, symbol Connector:Conn_01x04_Socket
- removed TP201, TP202, TP203: TestPoint, TestPoint:TestPoint_Pad_D1.0mm, symbol Connector:TestPoint
- added C203: 1n, Capacitor_SMD:C_1206_3216Metric, symbol Device:C_Small
- added C204, C205: 100n, Capacitor_SMD:C_0402_1005Metric, symbol Device:C_Small
- added R201: 1M, Resistor_SMD:R_2010_5025Metric, symbol Device:R
- added R202: 100, Resistor_SMD:R_0402_1005Metric, symbol Device:R_Small
- added SW201: TS50810-411-02528, lcsc_lib:SW-SMD_L6.2-W3.7-LS8.0, symbol lcsc_lib:TS50810-411-02528
- added U202: ETH, lcsc_lib:RJ45-SMD_HR963380AE, symbol lcsc_lib:HR963380AE
- renumbered U202 to U203
Connections:
- net Ethernet_Pair0_N: now also U202.2
- net Ethernet_Pair0_P: now also U202.1
- net Ethernet_Pair1_N: now also U202.4
- net Ethernet_Pair1_P: now also U202.3
- net Ethernet_Pair2_N: now also U202.8
- net Ethernet_Pair2_P: now also U202.7
- net Ethernet_Pair3_N: now also U202.10
- net Ethernet_Pair3_P: now also U202.9
- net GND: now also C204.2, C205.2, R201.1, SW201.2
- net MASKROM_KEY: now also R202.1
- net UART4_RX_M1: now reaches U201.24 (GPIO26)
- net UART0_TX_M0: now reaches U201.89 (WiFi_nDisable)
- net UART0_RTSN: now reaches U201.91 (BT_nDisable)
- net CAN0_RX_M1: no longer names the net of U201.57 (SD_CLK)
- net CAN0_TX_M1: no longer names the net of U201.62 (SD_CMD)
- net CAN1_RX_M1: no longer names the net of U201.31 (GPIO12)
- net CAN1_TX_M1: no longer names the net of U201.21 (PI_nLED_Activity)
- net I2C8_SCL_M0: no longer names the net of U201.69 (SD_DAT2)
- net I2C8_SDA_M0: no longer names the net of U201.61 (SD_DAT3)
- net UART3_CTSN_1V8: no longer names the net of U201.46 (GPIO22)
- net UART3_RTSN_1V8 renamed SPI4_CLK_M0_1V8
- net UART4_CTSN_1V8: no longer names the net of U201.34 (GPIO5)
- new net: R202.2, SW201.1
- new net: C203.1, R201.2
- new net CT0: C204.1, U202.5
- new net CT1: C205.1, U202.6
- new net Earth: C203.2, U202.15
- no-connect marks 44 -> 52
Other:
- moved on the sheet: C201, C202
