File: electrical/motion_control/board/cm5-u13b.kicad_sch (KiCad schematic)
At the start: 2 parts, among them J301 USB_MASKROM, U301 Hirose DF40C-100DS-0.4V

Commit message: new boards, new device tree image
Parts:
- removed J301: USB_MASKROM, Connector_JST:JST_GH_SM04B-GHS-TB_1x04-1MP_P1.25mm_Horizontal, symbol Connector:Conn_01x04_Socket
- added R301, R302: 5.1k, Resistor_SMD:R_0402_1005Metric, symbol Device:R_Small
- added USB301: TYPE-C 16PIN 2MD, lcsc_lib:USB-C-SMD_TYPE-C-16PIN-2MD-073, symbol lcsc_lib:TYPE-C16PIN2MD
Connections:
- net GND: now also R301.1, R302.1, USB301.A1B12 (GND), USB301.B1A12 (GND)
- net USB2_D+: now also USB301.A6 (Dp1), USB301.B6 (Dp2)
- net USB2_D-: now also USB301.A7 (Dn1), USB301.B7 (Dn2)
- net UART4_TX_M1: now reaches U301.109 (PCIe_nRST)
- new net: R302.2, USB301.B5 (CC2)
- new net: R301.2, USB301.A5 (CC1)
- no-connect marks 68 -> 73
