File: electrical/motion_control/board/spi-can.kicad_sch (KiCad schematic)
At the start: 25 parts, among them J601 SPI00_CAN_OUT, J602 SPI01_CAN_OUT, J603 SPI02_CAN_OUT, U501 MCP2518FD-xQBB, U502 MCP2518FD-xQBB, U503 MCP2518FD-xQBB, U602 TXB0104PW, U603 SN65HVD230, U606 SN65HVD230, U607 SN65HVD230, Y601 40M, Y602 40M, Y603 40M

Commit message: new boards, new device tree image
Parts:
- removed C603: 100n, Capacitor_SMD:C_0402_1005Metric, symbol Device:C_Small
- removed J601: SPI00_CAN_OUT, Connector_JST:JST_GH_SM02B-GHS-TB_1x02-1MP_P1.25mm_Horizontal, symbol Connector:Conn_01x02_Pin
- removed J602: SPI01_CAN_OUT, Connector_JST:JST_GH_SM02B-GHS-TB_1x02-1MP_P1.25mm_Horizontal, symbol Connector:Conn_01x02_Pin
- removed J603: SPI02_CAN_OUT, Connector_JST:JST_GH_SM02B-GHS-TB_1x02-1MP_P1.25mm_Horizontal, symbol Connector:Conn_01x02_Pin
- removed R602: 10k, Resistor_SMD:R_0402_1005Metric, symbol Device:R_Small
- removed U602: TXB0104PW, Package_SO:TSSOP-14_4.4x5mm_P0.65mm, symbol Logic_LevelTranslator:TXB0104PW
- added C601, C608, C609, C611, C612: 20p, Capacitor_SMD:C_0603_1608Metric, symbol Device:C_Small
- added R601, R605, R606: 120, Resistor_SMD:R_0402_1005Metric, symbol Device:R_Small
- added U601, U608, U609: MCP2518FD-xQBB, Package_SO:SOIC-14_3.9x8.7mm_P1.27mm, symbol Interface_CAN_LIN:MCP2518FD-xQBB
- added U604, U611, U612: SN65HVD230, Package_SO:SOIC-8_3.9x4.9mm_P1.27mm, symbol Interface_CAN_LIN:SN65HVD230
- added Y601, Y605, Y606: 40M, Crystal:Crystal_SMD_3225-4Pin_3.2x2.5mm, symbol Device:Crystal_GND24
- C604: value 100n -> 20p; footprint Capacitor_SMD:C_0402_1005Metric -> Capacitor_SMD:C_0603_1608Metric; LCSC C77020 -> C165732
- renumbered C601 to C602, C606 to C603, C602 to C605, C608 to C606, C605 to C607, C607 to C610, R601 to R602, R605 to R603, U501 to U602, U503 to U603, U603 to U605, U607 to U606, U502 to U607, U606 to U610, Y601 to Y602, Y602 to Y604
Connections:
- net +3V3: now also U601.14 (VDD), U604.3 (VCC), U608.14 (VDD), U609.14 (VDD), U611.3 (VCC), U612.3 (VCC); no longer C604.1
- net GND: now also C601.2, C608.2, C609.2, C611.2, C612.2, U601.15 (VSS), U601.7 (VSS), U604.2 (GND), U604.8 (Rs), U608.15 (VSS), U608.7 (VSS), U609.15 (VSS), U609.7 (VSS), U611.2 (GND), U611.8 (Rs), U612.2 (GND), U612.8 (Rs), Y601.2, Y601.4, Y605.2, Y605.4, Y606.2, Y606.4
- net SPI0_CLK: no longer U603.10 (SCK)
- net SPI0_SI: no longer U603.11 (SDI)
- net SPI0_SO: no longer U603.12 (SDO)
- net SPI00_CAN+ renamed CAN3+
- net SPI00_CAN- renamed CAN3-
- net SPI01_CAN+ renamed CAN0+
- net SPI01_CAN- renamed CAN0-
- net SPI02_CAN+ renamed CAN4+
- net SPI02_CAN- renamed CAN4-
- net SPI02_OSC_1 renamed SPI10_OSC_1
- net SPI02_OSC_2 renamed SPI10_OSC_2
- net SPI0_CS2 renamed SPI1_CS0
- net SPI0_INT2 renamed SPI1_INT0
- new net: U609.1 (TXCAN), U612.1 (D)
- new net: U609.2 (RXCAN), U612.4 (R)
- new net: U601.1 (TXCAN), U604.1 (D)
- new net: U601.2 (RXCAN), U604.4 (R)
- new net: U608.1 (TXCAN), U611.1 (D)
- new net: U608.2 (RXCAN), U611.4 (R)
- new net CAN1+: R605.1, U611.7 (CANH)
- new net CAN1-: R605.2, U611.6 (CANL)
- new net CAN2+: R606.1, U612.7 (CANH)
- new net CAN2-: R606.2, U612.6 (CANL)
- new net CAN5+: R601.1, U604.7 (CANH)
- new net CAN5-: R601.2, U604.6 (CANL)
- new net SPI11_OSC_1: C608.1, U608.6 (OSC1), Y605.1
- new net SPI11_OSC_2: C611.1, U608.5 (OSC2), Y605.3
- new net SPI1_CLK: U603.10 (SCK), U608.10 (SCK)
- new net SPI1_CS1: U608.13 (~{CS})
- new net SPI1_INT1: U608.4 (~{INT})
- new net SPI1_SI: U603.11 (SDI), U608.11 (SDI)
- new net SPI1_SO: U603.12 (SDO), U608.12 (SDO)
- new net SPI40_OSC_1: C601.1, U601.6 (OSC1), Y601.1
- new net SPI40_OSC_2: C604.1, U601.5 (OSC2), Y601.3
- new net SPI41_OSC_1: C609.1, U609.6 (OSC1), Y606.1
- new net SPI41_OSC_2: C612.1, U609.5 (OSC2), Y606.3
- new net SPI4_CLK: U601.10 (SCK), U609.10 (SCK)
- new net SPI4_CS0: U601.13 (~{CS})
- new net SPI4_CS1: U609.13 (~{CS})
- new net SPI4_INT0: U601.4 (~{INT})
- new net SPI4_INT1: U609.4 (~{INT})
- new net SPI4_SI: U601.11 (SDI), U609.11 (SDI)
- new net SPI4_SO: U601.12 (SDO), U609.12 (SDO)
- no-connect marks 11 -> 24
Other:
- note added: "### OSCILLATOR DECOUPLING CAPACITANCE CALCULATION ### C_L = (C**2 / 2C) + C_S C_L = load capacitance C_S = stray capacitance C = decoupling capacitance Assume C_L = 15p, C_S = 5p, 2C * 10p = C**2 20p * C = C**2 C = 20p Choosing 20p, closest value available"
- note removed: "C_L = (C**2 / 2C) + C_S C_L = load capacitance C_S = stray capacitance C = decoupling capacitance Assume C_L = 15p, C_S = 5p, 2C * 10p = C**2 20p * C = C**2 C = 20p Choosing 20p, closest value available"
- moved on the sheet: C602, C603, C605, C606, R602, R603, U602, U603, U605, U606, Y602, Y603
