Commit message: sim-model: update pelvis_link mass properties for ASV1_200_02A 6061-T6
ASV1_200_02A was re-specified in SolidWorks from 7075-T6 to 6061-T6.
Density falls 3.9% (2810 -> 2700 kg/m3) at unchanged geometry, so the
component loses 2.393 g and pelvis_link's mass, centre of mass and
inertia tensor all move with it.

  mass  3.506912512 -> 3.5045195956408359 kg

Re-exported mass properties applied to both models that carry them, so
the URDF and the MJCF do not disagree about the same link:

  sim-model/urdf/asimov_1.urdf   <inertial> origin, mass, inertia
  sim-model/xmls/asimov_1.xml    <inertial> pos, mass, fullinertia

Mesh geometry is untouched - no STL or STEP changes in this branch.
REQ-L0-MASS measures the MJCF mass sum and stays inside its 35 kg
limit; test_total_link_mass_is_within_the_l0_budget re-verifies it.

Co-Authored-By: Claude Opus 5 <noreply@anthropic.com>

File: sim-model/urdf/asimov_1.urdf (robot description, URDF)
Before this commit: robot asimov_1, 26 links, 25 joints
Links:
- link pelvis_link: mass 3.506912512 -> 3.5045195956408359
